File: displayboard/displayboard/displayboard.kicad_sch (KiCad schematic)
At the start: 1 part, among them SW1 RotaryEncoder_Switch

Commit message: V1.2
Parts:
- added C1, C2: C_Small, Capacitor_SMD:C_0805_2012Metric, symbol Device:C_Small
Connections:
- net ADC0_GP26: now also C1.1
- net ADC1_GP27: now also C2.1
- net AGND: now also C1.2, C2.2
Changed lines of the file:
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@@
 	(paper "A4")
+	(junction
+		(at 102.87 64.77)
+		(diameter 0)
+		(color 0 0 0 0)
+	)
+	(junction
+		(at 92.71 68.58)
+		(diameter 0)
+		(color 0 0 0 0)
+	)
+	(junction
+		(at 87.63 54.61)
+		(diameter 0)
+		(color 0 0 0 0)
+	)
+	(junction
+		(at 92.71 59.69)
+		(diameter 0)
+		(color 0 0 0 0)
+	)
 	(junction
 		(at 118.11 60.96)
@@
 	(wire
 		(pts
-			(xy 93.98 54.61) (xy 100.33 54.61)
+			(xy 86.36 54.61) (xy 87.63 54.61)
 		)
 		(stroke
@@
 	(wire
 		(pts
+			(xy 92.71 68.58) (xy 102.87 68.58)
+		)
+		(stroke
+			(width 0)
+			(type default)
+		)
+	)
+	(wire
+		(pts
+			(xy 92.71 59.69) (xy 100.33 59.69)
+		)
+		(stroke
+			(width 0)
+			(type default)
+		)
+	)
+	(wire
+		(pts
+			(xy 102.87 64.77) (xy 118.11 64.77)
+		)
+		(stroke
+			(width 0)
+			(type default)
+		)
+	)
+	(wire
+		(pts
 			(xy 96.52 57.15) (xy 96.52 64.77)
 		)
@@
 	(wire
 		(pts
+			(xy 87.63 68.58) (xy 92.71 68.58)
+		)
+		(stroke
+			(width 0)
+			(type default)
+		)
+	)
+	(wire
+		(pts
 			(xy 115.57 59.69) (xy 118.11 59.69)
 		)
@@
 	(wire
 		(pts
-			(xy 96.52 64.77) (xy 118.11 64.77)
+			(xy 87.63 54.61) (xy 100.33 54.61)
+		)
+		(stroke
+			(width 0)
+			(type default)
+		)
+	)
+	(wire
+		(pts
+			(xy 96.52 64.77) (xy 102.87 64.77)
+		)
+		(stroke
+			(width 0)
+			(type default)
+		)
+	)
+	(wire
+		(pts
+			(xy 102.87 68.58) (xy 102.87 64.77)
 		)
 		(stroke
@@
 	(wire
 		(pts
-			(xy 93.98 59.69) (xy 100.33 59.69)
+			(xy 86.36 59.69) (xy 92.71 59.69)
 		)
 		(stroke
@@
 		(pts
 			(xy 118.11 59.69) (xy 118.11 60.96)
+		)
+		(stroke
+			(width 0)
+			(type default)
+		)
+	)
+	(wire
+		(pts
+			(xy 87.63 54.61) (xy 87.63 63.5)
+		)
+		(stroke
+			(width 0)
+			(type default)
+		)
+	)
+	(wire
+		(pts
+			(xy 92.71 59.69) (xy 92.71 63.5)
 		)
 		(stroke
@@
 	(global_label "ADC1_GP27"
 		(shape input)
-		(at 93.98 59.69 180)
+		(at 86.36 59.69 180)
 		(fields_autoplaced yes)
 		(effects
@@
 		)
 		(property "Intersheetrefs" "${INTERSHEET_REFS}"
-			(at 80.2301 59.69 0)
+			(at 72.6101 59.69 0)
 			(effects
 				(font
@@
 	(global_label "ADC0_GP26"
 		(shape input)
-		(at 93.98 54.61 180)
+		(at 86.36 54.61 180)
 		(fields_autoplaced yes)
 		(effects
@@
 		)
 		(property "Intersheetrefs" "${INTERSHEET_REFS}"
-			(at 80.2301 54.61 0)
+			(at 72.6101 54.61 0)
 			(effects
 				(font
@@
 			)
 		)
+	)
+	(symbol
+		(lib_id "Device:C_Small")
+		(at 92.71 66.04 0)
+		(unit 1)
+		(exclude_from_sim no)
+		(in_bom yes)
+		(on_board yes)
+		(dnp no)
+		(property "Reference" "C2"
+			(at 91.694 71.882 0)
+			(effects
+				(font
+					(size 1.27 1.27)
+				)
+				(justify left)
+			)
+		)
+		(property "Value" "C_Small"
+			(at 94.996 71.882 0)
+			(effects
+				(font
+					(size 1.27 1.27)
+				)
+				(justify left)
+			)
+		)
+		(property "Footprint" "Capacitor_SMD:C_0805_2012Metric"
+			(at 92.71 66.04 0)
+			(effects
+				(font
+					(size 1.27 1.27)
+				)
+				(hide yes)
+			)
+		)
+		(property "Datasheet" "~"
+			(at 92.71 66.04 0)
+			(effects
+				(font
+					(size 1.27 1.27)
+				)
+				(hide yes)
+			)
+		)
+		(property "Description" "Unpolarized capacitor, small symbol"
+			(at 92.71 66.04 0)
+			(effects
+				(font
+					(size 1.27 1.27)
+				)
+				(hide yes)
+			)
+		)
+		(pin "1"
+		)
+		(pin "2"
+		)
+		(instances
+			(project "displayboard"
+				(path "/7d4007be-7c30-4eeb-bece-b3e563eb9368"
+					(reference "C2")
+					(unit 1)
+				)
+			)
+		)
+	)
+	(symbol
+		(lib_id "Device:C_Small")
+		(at 87.63 66.04 0)
+		(unit 1)
+		(exclude_from_sim no)
+		(in_bom yes)
+		(on_board yes)
+		(dnp no)
+		(property "Reference" "C1"
+			(at 77.724 65.786 0)
+			(effects
+				(font
+					(size 1.27 1.27)
+				)
+				(justify left)
+			)
+		)
+		(property "Value" "C_Small"
+			(at 74.168 68.834 0)
+			(effects
+				(font
+					(size 1.27 1.27)
+				)
+				(justify left)
+			)
+		)
+		(property "Footprint" "Capacitor_SMD:C_0805_2012Metric"
+			(at 87.63 66.04 0)
+			(effects
+				(font
+					(size 1.27 1.27)
+				)
+				(hide yes)
+			)
+		)
+		(property "Datasheet" "~"
+			(at 87.63 66.04 0)
+			(effects
+				(font
+					(size 1.27 1.27)
+				)
+				(hide yes)
+			)
+		)
+		(property "Description" "Unpolarized capacitor, small symbol"
+			(at 87.63 66.04 0)
+			(effects
+				(font
+					(size 1.27 1.27)
+				)
+				(hide yes)
+			)
+		)
+		(pin "1"
+		)
+		(pin "2"
+		)
+		(instances
+			(project ""
+				(path "/7d4007be-7c30-4eeb-bece-b3e563eb9368"
+					(reference "C1")
+					(unit 1)
+				)
+			)
+		)
