File: mainboard.kicad_pcb (KiCad board)
At the start: 2 copper layers, 157.6 x 135.8 mm, 67 parts, among them J1 DRV8833-1, J13 Conn_PCA9685, J14 Conn_01x02, J15 Conn_01x02, J16 Conn_01x02, J18 Screw_Terminal_01x06, J19 Screw_Terminal_01x06, J2 DRV8833-0, J20 Screw_Terminal_01x06, J21 Screw_Terminal_01x06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

Commit message: Ready boards
powerboard, displayboard and mainboard all ready to mill
Parts:
- moved C1 6.83 mm to (294.0, 95.8), turned to 45 degrees
- moved C1 2.41 mm to (295.7, 97.5)
- moved REF** 1.56 mm to (352.4, 52.0)
- moved ? 0.45 mm to (383.2, 96.4)
- moved ? 0.07 mm to (289.9, 86.4)
Routing:
- net 5V_BUCK: track 348.2 -> 343.4 mm
- net TOTEM-EXTEND: track 90.7 -> 86.4 mm
- net SORT(en/dis): track 58.8 -> 60.6 mm, vias 2 -> 3
- net PCA9685_SCL: track 67.2 -> 68.2 mm
- net PCA9685_SDA: track 65.5 -> 66.3 mm
- net PIC_STATE: track 42.4 -> 43.1 mm
- net 12V_BUCK2: track 127.4 -> 126.8 mm
- added copper zone on B.Cu, net 5V_BUCK
Other:
- outline, holes or cut-outs redrawn
- board text added: "-+"
- board text added: "F(L)"
- board text added: "F(R)"
- board text added: "R(L)"
- board text added: "R(R)"
- board text removed: "FRONT(L)"
- board text removed: "FRONT(R)"
- board text removed: "REAR(L)"
- board text removed: "REAR(R)"
